Commit message: cross entropy with position control

File: gym_gazebo/envs/ros_ws/src/wheel_gazebo/urdf/wheel.urdf (robot description, URDF)
Before this commit: robot onshape, 4 links, 3 joints
Joints:
- joint rev: limit effort=20 velocity=20 -> effort=1 velocity=20

Commit message: gazebo replacing cam

File: gym_gazebo/envs/ros_ws/src/wheel_gazebo/urdf/wheel.urdf (robot description, URDF)
Before this commit: robot onshape, 4 links, 3 joints
Links:
- link base_link: geometry collision mesh filename=file:///home/mackenzie/gym-gazebo-noetic/gym_gazebo/envs/ro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; visual mesh filename=file:///home/mackenzie/gym-gazebo-noetic/gym_gazebo/envs/ro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
- link wheel: geometry collision mesh filename=file:///home/mackenzie/gym-gazebo-noetic/gym_gazebo/envs/ro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; visual mesh filename=file:///home/mackenzie/gym-gazebo-noetic/gym_gazebo/envs/ro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

Commit message: WIP Gazebo vs Camera Training delay decreased

File: gym_gazebo/envs/ros_ws/src/wheel_gazebo/urdf/wheel.urdf (robot description, URDF)
Before this commit: robot onshape, 4 links, 3 joints
Joints:
- joint camera_joint: origin xyz=0 1 .3 rpy=0 0 -1.57079632679 -> xyz=0 0.5 .3 rpy=0 0 -1.57079632679

Commit message: Training with examples/gazebo_wheel/gazebo_wheel_ex.py showing learning

File: gym_gazebo/envs/ros_ws/src/wheel_gazebo/urdf/wheel.urdf (robot description, URDF)
Before this commit: robot onshape, 4 links, 3 joints
Links:
- link base_link: geometry collision mesh filename=file:///home/seanghaeli/gym-gazebo-noetic/gym_gazebo/envs/r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; visual mesh filename=file:///home/seanghaeli/gym-gazebo-noetic/gym_gazebo/envs/r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
- link wheel: geometry collision mesh filename=file:///home/seanghaeli/gym-gazebo-noetic/gym_gazebo/envs/r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; visual mesh filename=file:///home/seanghaeli/gym-gazebo-noetic/gym_gazebo/envs/r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

Commit message: Made the ball black. Quantify sim time delays.

File: gym_gazebo/envs/ros_ws/src/wheel_gazebo/urdf/wheel.urdf (robot description, URDF)
Before this commit: robot onshape, 4 links, 3 joints
Links:
- link base_link: geometry collision mesh filename=file:///home/fizzer/Documents/Capstone/gym-gazebo-noetic/gy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; visual mesh filename=file:///home/fizzer/Documents/Capstone/gym-gazebo-noetic/gy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
- link wheel: geometry collision mesh filename=file:///home/fizzer/Documents/Capstone/gym-gazebo-noetic/gy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; visual mesh filename=file:///home/fizzer/Documents/Capstone/gym-gazebo-noetic/gy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

Commit message: training with camera subscribing (not working

File: gym_gazebo/envs/ros_ws/src/wheel_gazebo/urdf/wheel.urdf (robot description, URDF)
Before this commit: robot onshape, 4 links, 3 joints
Links:
- link base_link: geometry collision mesh filename=file:///home/fizzer/Documents/Capstone/gym-gazebo-noetic/gy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; visual mesh filename=file:///home/fizzer/Documents/Capstone/gym-gazebo-noetic/gy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
- link wheel: geometry collision mesh filename=file:///home/fizzer/Documents/Capstone/gym-gazebo-noetic/gy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; visual mesh filename=file:///home/fizzer/Documents/Capstone/gym-gazebo-noetic/gy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

File: gym_gazebo/envs/ros_ws/src/wheel_gazebo/urdf/wheel_orig.urdf (robot description, URDF)
Before this commit: robot onshape, 3 links, 2 joints
Links:
- link base_link: geometry collision mesh filename=file:///home/fizzer/Documents/Capstone/catkin_ws/src/wheel_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; visual mesh filename=file:///home/fizzer/Documents/Capstone/catkin_ws/src/wheel_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
- link wheel: geometry collision mesh filename=file:///home/fizzer/Documents/Capstone/catkin_ws/src/wheel_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; visual mesh filename=file:///home/fizzer/Documents/Capstone/catkin_ws/src/wheel_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

Commit message: negative log likelihood loss training attempt

File: gym_gazebo/envs/ros_ws/src/wheel_gazebo/urdf/wheel.urdf (robot description, URDF)
Before this commit: robot onshape, 4 links, 3 joints
Links:
- link base_link: geometry collision mesh filename=file:///home/seanghaeli/gym-gazebo-noetic/gym_gazebo/envs/r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; visual mesh filename=file:///home/seanghaeli/gym-gazebo-noetic/gym_gazebo/envs/r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
- link wheel: geometry collision mesh filename=file:///home/seanghaeli/gym-gazebo-noetic/gym_gazebo/envs/r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; visual mesh filename=file:///home/seanghaeli/gym-gazebo-noetic/gym_gazebo/envs/r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

File: gym_gazebo/envs/ros_ws/src/wheel_gazebo/urdf/wheel_orig.urdf (robot description, URDF)
Before this commit: robot onshape, 3 links, 2 joints
Links:
- link base_link: geometry collision mesh filename=file:///home/seanghaeli/catkin_ws/src/wheel_gazebo/urdf/bas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; visual mesh filename=file:///home/seanghaeli/catkin_ws/src/wheel_gazebo/urdf/bas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
- link wheel: geometry collision mesh filename=file:///home/seanghaeli/catkin_ws/src/wheel_gazebo/urdf/whe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; visual mesh filename=file:///home/seanghaeli/catkin_ws/src/wheel_gazebo/urdf/whe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
