Commit message: WIP: Coverleaf PID even possible?? not so far...

File: gym_gazebo/envs/ros_ws/src/wheel_gazebo/urdf/clover/clover.urdf (robot description, URDF)
Before this commit: robot onshape, 4 links, 3 joints
Links:
- link wheel: mass 0.331756 -> 0.331752

Commit message: minor: fix angle offset

File: gym_gazebo/envs/ros_ws/src/wheel_gazebo/urdf/clover/clover.urdf (robot description, URDF)
Before this commit: robot onshape, 4 links, 3 joints
Joints:
- joint rev: origin xyz=-7.60623e-18 -3.5982e-17 0.2032 rpy=1.5708 -0.868659 3.14159 -> xyz=-6.0648e-18 -1.61908e-17 0.2032 rpy=-1.5708 1.5708 0
