Commit message: WIP: Branch rename

File: gym_gazebo/envs/ros_ws/src/wheel_gazebo/urdf/peanut/robot.urdf (robot description, URDF)
Before this commit: robot onshape, 4 links, 3 joints
Links:
- link base_link: mass 11.195 -> 11.8457
- link wheel: mass 0.190419 -> 0.742847
Joints:
- joint rev: origin xyz=-3.46945e-18 -1.61908e-17 0.2032 rpy=1.5708 2.77556e-17 3.14159 -> xyz=-5.55112e-17 -1.61908e-17 0.2794 rpy=1.5708 6.12323e-17 -3.14159
